Commit message: base_link added and removed z-offset from world from the robot base (stand)

File: optimo_description/urdf/optimo.xacro (robot description, xacro)
@@ -45,5 +45,5 @@
                 <parent link="world" />
                 <child link="${prefix}stand" />
-                <origin xyz="0 0 1" rpy="0 0 -1.57" />
+                <origin xyz="0 0 0" rpy="0 0 0" />
             </joint>
             <link name="${prefix}stand">
@@ -51,5 +51,5 @@
                     <origin xyz="0 0 -0.5" rpy="0 0 0" />
                     <geometry>
-                        <box size="0.3 0.3 1" />
+                        <box size="0.5 0.5 1" />
                     </geometry>
                     <material name="white" />
@@ -58,10 +58,16 @@
                     <origin xyz="0 0 -0.5" rpy="0 0 0" />
                     <geometry>
-                        <box size="0.3 0.3 1" />
+                        <box size="0.5 0.5 1" />
                     </geometry>
                 </collision>
             </link>
-            <joint name="${prefix}stand_to_link0" type="fixed">
+            <joint name="${prefix}stand_to_base_link" type="fixed">
                 <parent link="${prefix}stand" />
+                <child link="${prefix}base_link" />
+                <origin xyz="0 0 0" rpy="0 0 0" />
+            </joint>
+            <link name="${prefix}base_link"/>
+            <joint name="${prefix}base_link_to_link0" type="fixed">
+                <parent link="${prefix}base_link" />
                 <child link="${prefix}link0" />
                 <!-- .27 puts the link on the stand -->
